Commit message: changed dimensions and wrote proper code for other stuff

File: simulation_ws/src/m2wr_description/urdf/m2wr.xacro (robot description, xacro)
@@ -9,10 +9,10 @@
     <inertial>
       <mass value="5"/>
-      <origin rpy="0 0 0" xyz="0 0 0.1"/>
-      <inertia ixx="0.0395416666667" ixy="0" ixz="0" iyy="0.106208333333" iyz="0" izz="0.106208333333"/>
+      <origin rpy="0 0 0" xyz="0 0 0"/>
+      <xacro:box_inertia m="5" x="0.12" y="0.08" z="0.03" />
     </inertial>
     <collision name="collision_chassis">
       <geometry>
-        <box size="0.5 0.3 0.07"/>
+        <box size="0.12 0.08 0.03"/>
       </geometry>
     </collision>
@@ -20,13 +20,18 @@
       <origin rpy="0 0 0" xyz="0 0 0"/>
       <geometry>
-        <box size="0.5 0.3 0.07"/>
+        <box size="0.12 0.08 0.03"/>
       </geometry>
       <material name="blue"/>
     </visual>
+    <inertial name="caster_fron_inertial">
+      <mass value="1"/>
+      <origin rpy="0 0 0" xyz="0 0 0"/>
+      <xacro:sphere_inertia m="1" r="0.015" />
+    </inertial>
     <!-- caster front -->
     <collision name="caster_front_collision">
-      <origin rpy=" 0 0 0" xyz="0.35 0 -0.05"/>
+      <origin rpy=" 0 0 0" xyz="0.04 0 -0.02"/>
       <geometry>
-        <sphere radius="0.05"/>
+        <sphere radius="0.015"/>
       </geometry>
       <surface>
@@ -37,4 +42,6 @@
             <slip1>1.0</slip1>
             <slip2>1.0</slip2>
+             <fdir1>0 1.0 0</fdir1>
+        <implicit_spring_damper>true</implicit_spring_damper>
           </ode>
         </friction>
@@ -42,7 +49,7 @@
     </collision>
     <visual name="caster_front_visual">
-      <origin rpy=" 0 0 0" xyz="0.2 0 -0.05"/>
+      <origin rpy=" 0 0 0" xyz="0.04 0 -0.02"/>
       <geometry>
-        <sphere radius="0.05"/>
+        <sphere radius="0.015"/>
       </geometry>
     </visual>
@@ -51,9 +58,9 @@
   <xacro:link_wheel name="link_left_wheel" />
   <!--   Joint for right wheel  -->
-  <xacro:joint_wheel name="joint_right_wheel"  child="link_right_wheel"  origin_xyz="-0.05 0.15 0"  />>
+  <xacro:joint_wheel name="joint_right_wheel"  child="link_right_wheel"  origin_xyz="-0.04 -0.04 0"  />>
   <!-- Left Wheel link -->
   <xacro:link_wheel name="link_right_wheel" />
   <!--   Joint for left wheel  -->
-  <xacro:joint_wheel name="joint_left_wheel"   child="link_left_wheel"   origin_xyz="-0.05 -0.15 0"  />
+  <xacro:joint_wheel name="joint_left_wheel"   child="link_left_wheel"   origin_xyz="-0.04 0.04 0"  />
    <link name="sensor_laser">
     <inertial>
@@ -61,10 +68,10 @@
       <mass value="1" />
       <!-- RANDOM INERTIA BELOW -->
-      <xacro:cylinder_inertia mass="1" r="0.05" l="0.1" />
+      <xacro:cylinder_inertia mass="1" r="0.01" l="0.03" />
     </inertial>
     <visual>
       <origin xyz="0 0 0" rpy="0 0 0" />
       <geometry>
-        <cylinder radius="0.05" length="0.1"/>
+        <cylinder radius="0.01" length="0.03"/>
       </geometry>
       <material name="white" />
@@ -73,10 +80,10 @@
       <origin xyz="0 0 0" rpy="0 0 0"/>
       <geometry>
-        <cylinder radius="0.05" length="0.1"/>
+        <cylinder radius="0.01" length="0.03"/>
       </geometry>
     </collision>
   </link>
   <joint name="joint_sensor_laser" type="fixed">
-    <origin xyz="0.15 0 0.05" rpy="0 0 0"/>
+    <origin xyz="0.04 0 0.03" rpy="0 0 0"/>
     <parent link="link_chassis"/>
     <child link="sensor_laser"/>

File: simulation_ws/src/m2wr_description/urdf/macro.xacro (robot description, xacro)
@@ -6,10 +6,10 @@
           <mass value="0.2"/>
           <origin rpy="0 1.5707 1.5707" xyz="0 0 0"/>
-          <inertia ixx="0.000526666666667" ixy="0" ixz="0" iyy="0.000526666666667" iyz="0" izz="0.001"/>
+          <xacro:cylinder_inertia mass="0.2" r="0.035" l="0.02" />
         </inertial>
         <collision name="link_right_wheel_collision">
           <origin rpy="0 1.5707 1.5707" xyz="0 0 0"/>
           <geometry>
-            <cylinder length="0.04" radius="0.1"/>
+            <cylinder length="0.02" radius="0.035"/>
           </geometry>
         </collision>
@@ -17,5 +17,5 @@
           <origin rpy="0 1.5707 1.5707" xyz="0 0 0"/>
           <geometry>
-            <cylinder length="0.04" radius="0.1"/>
+            <cylinder length="0.02" radius="0.035"/>
           </geometry>
         </visual>
@@ -36,3 +36,13 @@
                 iyy="${mass*(3*r*r+l*l)/12}" iyz = "0" izz="${mass*(r*r)/2}" />
 </xacro:macro>
+<xacro:macro name="box_inertia" params="m x y z">
+        <inertia  ixx="${m*(y*y+z*z)/12}" ixy = "0" ixz = "0"
+                  iyy="${m*(x*x+z*z)/12}" iyz = "0"
+                  izz="${m*(x*x+z*z)/12}" />
+</xacro:macro>
+<xacro:macro name="sphere_inertia" params="m r">
+        <inertia  ixx="${2*m*r*r/5}" ixy = "0" ixz = "0"
+                  iyy="${2*m*r*r/5}" iyz = "0"
+                  izz="${2*m*r*r/5}" />
+</xacro:macro>
 </robot>

Commit message: wall follower for mazemapping added

File: simulation_ws/src/m2wr_description/urdf/m2wr.xacro (robot description, xacro)
@@ -27,11 +27,11 @@
       <mass value="1"/>
       <origin rpy="0 0 0" xyz="0 0 0"/>
-      <xacro:sphere_inertia m="1" r="0.015" />
+      <xacro:sphere_inertia m="1" r="0.005" />
     </inertial>
-    <!-- caster front -->
+    caster front
     <collision name="caster_front_collision">
-      <origin rpy=" 0 0 0" xyz="0.04 0 -0.02"/>
+      <origin rpy=" 0 0 0" xyz="0.04 0 -0.015"/>
       <geometry>
-        <sphere radius="0.015"/>
+        <sphere radius="0.005"/>
       </geometry>
       <surface>
@@ -49,7 +49,7 @@
     </collision>
     <visual name="caster_front_visual">
-      <origin rpy=" 0 0 0" xyz="0.04 0 -0.02"/>
+      <origin rpy=" 0 0 0" xyz="0.04 0 -0.015"/>
       <geometry>
-        <sphere radius="0.015"/>
+        <sphere radius="0.005"/>
       </geometry>
     </visual>
@@ -68,10 +68,10 @@
       <mass value="1" />
       <!-- RANDOM INERTIA BELOW -->
-      <xacro:cylinder_inertia mass="1" r="0.01" l="0.03" />
+      <xacro:cylinder_inertia mass="1" r="0.01" l="0.02" />
     </inertial>
     <visual>
       <origin xyz="0 0 0" rpy="0 0 0" />
       <geometry>
-        <cylinder radius="0.01" length="0.03"/>
+        <cylinder radius="0.01" length="0.02"/>
       </geometry>
       <material name="white" />
@@ -80,10 +80,10 @@
       <origin xyz="0 0 0" rpy="0 0 0"/>
       <geometry>
-        <cylinder radius="0.01" length="0.03"/>
+        <cylinder radius="0.01" length="0.02"/>
       </geometry>
     </collision>
   </link>
   <joint name="joint_sensor_laser" type="fixed">
-    <origin xyz="0.04 0 0.03" rpy="0 0 0"/>
+    <origin xyz="-0.04 0 0.025" rpy="0 0 0"/>
     <parent link="link_chassis"/>
     <child link="sensor_laser"/>

File: simulation_ws/src/m2wr_description/urdf/macro.xacro (robot description, xacro)
@@ -6,10 +6,10 @@
           <mass value="0.2"/>
           <origin rpy="0 1.5707 1.5707" xyz="0 0 0"/>
-          <xacro:cylinder_inertia mass="0.2" r="0.035" l="0.02" />
+          <xacro:cylinder_inertia mass="0.2" r="0.02" l="0.02" />
         </inertial>
         <collision name="link_right_wheel_collision">
           <origin rpy="0 1.5707 1.5707" xyz="0 0 0"/>
           <geometry>
-            <cylinder length="0.02" radius="0.035"/>
+            <cylinder length="0.02" radius="0.02"/>
           </geometry>
         </collision>
@@ -17,5 +17,5 @@
           <origin rpy="0 1.5707 1.5707" xyz="0 0 0"/>
           <geometry>
-            <cylinder length="0.02" radius="0.035"/>
+            <cylinder length="0.02" radius="0.02"/>
           </geometry>
         </visual>
